Commit message: edrone Initial Commit

File: rotors_description/urdf/component_snippets.xacro (robot description, xacro)
@@ -6,4 +6,6 @@
   Copyright 2015 Janosch Nikolic, ASL, ETH Zurich, Switzerland
   Copyright 2015 Markus Achtelik, ASL, ETH Zurich, Switzerland
+  Copyright 2018 Giuseppe Silano, University of Sannio in Benevento, Italy
+  Copyright 2018 Luigi Iannelli, University of Sannio in Benevento, Italy
   Licensed under the Apache License, Version 2.0 (the "License");
   you may not use this file except in compliance with the License.
@@ -28,5 +30,5 @@
         <frameId>${namespace}/base_link</frameId>
         <rotorVelocitySlowdownSim>${rotor_velocity_slowdown_sim}</rotorVelocitySlowdownSim>
-	<waitToRecordBag>${wait_to_record_bag}</waitToRecordBag>
+  <waitToRecordBag>${wait_to_record_bag}</waitToRecordBag>
       </plugin>
     </gazebo>
@@ -250,6 +252,6 @@
   <!-- =============================================================== -->
   <!-- <xacro:macro
-  		name="ros_interface_plugin_macro"
-  		params="namespace">
+      name="ros_interface_plugin_macro"
+      params="namespace">
     <gazebo>
       <plugin name="ros_interface_plugin" filename="librotors_gazebo_ros_interface_plugin.so">
@@ -269,18 +271,18 @@
       <plugin name="mavlink_interface" filename="librotors_gazebo_mavlink_interface.so">
         <robotNamespace>${namespace}</robotNamespace>
-	<mavlinkControlSubTopic>${mavlink_sub_topic}</mavlinkControlSubTopic>
+  <mavlinkControlSubTopic>${mavlink_sub_topic}</mavlinkControlSubTopic>
         <imuSubTopic>${imu_sub_topic}</imuSubTopic>
         <mavlinkHilSensorPubTopic>${mavlink_pub_topic}</mavlinkHilSensorPubTopic>
-	<motorSpeedsPubTopic>${motors_speeds_pub_topic}</motorSpeedsPubTopic>
-	<gpsUpdateFreq>${gps_update_freq}</gpsUpdateFreq> <!-- Frequency of HIL GPS messages [Hz] -->
-	<rotorCount>${rotor_count}</rotorCount>
+  <motorSpeedsPubTopic>${motors_speeds_pub_topic}</motorSpeedsPubTopic>
+  <gpsUpdateFreq>${gps_update_freq}</gpsUpdateFreq> <!-- Frequency of HIL GPS messages [Hz] -->
+  <rotorCount>${rotor_count}</rotorCount>
         <!-- [Gauss] Below are the North, East, and Down components of the Earth's magnetic field at the reference location.
              The default reference location is Zurich (lat=+47.3667degN, lon=+8.5500degE, h=+500m, WGS84).
-	     You can obtain the magnetic field strength for your location using the World Magnetic Model:
+       You can obtain the magnetic field strength for your location using the World Magnetic Model:
              https://www.ngdc.noaa.gov/geomag/WMM/calculators.shtml -->
         <referenceMagNorth>${reference_magnetic_field_north}</referenceMagNorth>
         <referenceMagEast>${reference_magnetic_field_east}</referenceMagEast>
         <referenceMagDown>${reference_magnetic_field_down}</referenceMagDown>
-	<referenceLatitude>${reference_latitude}</referenceLatitude> <!-- the initial latitude [degrees [-90, 90]] -->
+  <referenceLatitude>${reference_latitude}</referenceLatitude> <!-- the initial latitude [degrees [-90, 90]] -->
         <referenceLongitude>${reference_longitude}</referenceLongitude> <!-- the initial longitude [degrees [-180, 180]] -->
         <referenceAltitude>${reference_altitude}</referenceAltitude> <!-- the initial altitude [m] -->
@@ -291,6 +293,6 @@
   <xacro:macro name="imu_plugin_macro"
     params="namespace imu_suffix parent_link imu_topic
-      mass_imu_sensor gyroscope_noise_density gyroscope_random_walk
-      gyroscope_bias_correlation_time gyroscope_turn_on_bias_sigma
+      mass_imu_sensor measurement_divisor measurement_delay gyroscope_noise_density
+      gyroscope_random_walk gyroscope_bias_correlation_time gyroscope_turn_on_bias_sigma
       accelerometer_noise_density accelerometer_random_walk
       accelerometer_bias_correlation_time accelerometer_turn_on_bias_sigma
@@ -319,4 +321,6 @@
         <imuTopic>${imu_topic}</imuTopic> <!-- (string): name of the sensor output topic and prefix of service names (defaults to imu) -->
         <gyroscopeNoiseDensity>${gyroscope_noise_density}</gyroscopeNoiseDensity> <!-- Gyroscope noise density (two-sided spectrum) [rad/s/sqrt(Hz)] -->
+        <measurementDivisor>${measurement_divisor}</measurementDivisor> <!-- only every (seq % measurementDivisor) == 0 measurement is published [int] -->
+        <measurementDelay>${measurement_delay}</measurementDelay> <!-- time that measurement gets held back before it's published in [simulation cycles (int)] -->
         <gyroscopeRandomWalk>${gyroscope_random_walk}</gyroscopeRandomWalk> <!-- Gyroscope bias random walk [rad/s/s/sqrt(Hz)] -->
         <gyroscopeBiasCorrelationTime>${gyroscope_bias_correlation_time}</gyroscopeBiasCorrelationTime> <!-- Gyroscope bias correlation time constant [s] -->
@@ -487,5 +491,5 @@
         <!-- [Tesla] Below is the reference Earth's magnetic field at the reference location in NED frame.
              The default reference location is Zurich (lat=+47.3667degN, lon=+8.5500degE, h=+500m, WGS84).
-	     You can obtain the magnetic field strength for your location using the World Magnetic Model:
+       You can obtain the magnetic field strength for your location using the World Magnetic Model:
              http://www.ngdc.noaa.gov/geomag-web/#igrfwmm -->
         <refMagNorth>${ref_mag_north}</refMagNorth>
@@ -748,4 +752,6 @@
       parent_link="${namespace}/vi_sensor_link"
       imu_topic="imu"
+      measurement_delay="0"
+      measurement_divisor="1"
       mass_imu_sensor="0.015"
       gyroscope_noise_density="0.0003394"
@@ -768,4 +774,6 @@
       parent_link="${parent_link}"
       imu_topic="ground_truth/imu"
+      measurement_delay="0"
+      measurement_divisor="1"
       mass_imu_sensor="0.00001"
       gyroscope_noise_density="0.0"
@@ -818,5 +826,7 @@
       parent_link="${parent_link}"
       imu_topic="imu"
-      mass_imu_sensor="0.015"
+      measurement_delay="0"
+      measurement_divisor="1"
+      mass_imu_sensor="0.00001"
       gyroscope_noise_density="0.0003394"
       gyroscope_random_walk="0.000038785"
@@ -827,4 +837,88 @@
       accelerometer_bias_correlation_time="300.0"
       accelerometer_turn_on_bias_sigma="0.1960">
+      <inertia ixx="0.00001" ixy="0.0" ixz="0.0" iyy="0.00001" iyz="0.0" izz="0.00001" />
+      <origin xyz="0 0 0" rpy="0 0 0" />
+    </xacro:imu_plugin_macro>
+  </xacro:macro>
+  <xacro:macro name="crazyflie2_odometry" params="namespace parent_link">
+      <xacro:odometry_plugin_macro
+        namespace="${namespace}"
+        odometry_sensor_suffix=""
+        parent_link="${parent_link}"
+        pose_topic="pose"
+        pose_with_covariance_topic="pose_with_covariance"
+        position_topic="position"
+        transform_topic="transform"
+        odometry_topic="odometry"
+        parent_frame_id="world"
+        child_frame_id="${namespace}/base_link"
+        mass_odometry_sensor="0.00001"
+        measurement_divisor="10"
+        measurement_delay="0"
+        unknown_delay="0.0"
+        noise_normal_position="0 0 0"
+        noise_normal_quaternion="0 0 0"
+        noise_normal_linear_velocity="0 0 0"
+        noise_normal_angular_velocity="0 0 0"
+        noise_uniform_position="0 0 0"
+        noise_uniform_quaternion="0 0 0"
+        noise_uniform_linear_velocity="0 0 0"
+        noise_uniform_angular_velocity="0 0 0"
+        enable_odometry_map="false"
+        odometry_map=""
+        image_scale="">
+        <inertia ixx="0.00001" ixy="0.0" ixz="0.0" iyy="0.00001" iyz="0.0" izz="0.00001" /> <!-- [kg m^2] [kg m^2] [kg m^2] [kg m^2] [kg m^2] [kg m^2] -->
+        <origin xyz="0.0 0.0 0.0" rpy="0.0 0.0 0.0" />
+      </xacro:odometry_plugin_macro>
+  </xacro:macro>
+<xacro:macro name="edrone_odometry" params="namespace parent_link">
+      <xacro:odometry_plugin_macro
+        namespace="${namespace}"
+        odometry_sensor_suffix=""
+        parent_link="${parent_link}"
+        pose_topic="pose"
+        pose_with_covariance_topic="pose_with_covariance"
+        position_topic="position"
+        transform_topic="transform"
+        odometry_topic="odometry"
+        parent_frame_id="world"
+        child_frame_id="${namespace}/base_link"
+        mass_odometry_sensor="0.00001"
+        measurement_divisor="10"
+        measurement_delay="0"
+        unknown_delay="0.0"
+        noise_normal_position="0 0 0"
+        noise_normal_quaternion="0 0 0"
+        noise_normal_linear_velocity="0 0 0"
+        noise_normal_angular_velocity="0 0 0"
+        noise_uniform_position="0 0 0"
+        noise_uniform_quaternion="0 0 0"
+        noise_uniform_linear_velocity="0 0 0"
+        noise_uniform_angular_velocity="0 0 0"
+        enable_odometry_map="false"
+        odometry_map=""
+        image_scale="">
+        <inertia ixx="0.00001" ixy="0.0" ixz="0.0" iyy="0.00001" iyz="0.0" izz="0.00001" /> <!-- [kg m^2] [kg m^2] [kg m^2] [kg m^2] [kg m^2] [kg m^2] -->
+        <origin xyz="0.0 0.0 0.0" rpy="0.0 0.0 0.0" />
+      </xacro:odometry_plugin_macro>
+  </xacro:macro>
+  <xacro:macro name="crazyflie2_imu" params="namespace parent_link">
+    <!-- Mount an MPU-9250 IMU. -->
+    <xacro:imu_plugin_macro
+      namespace="${namespace}"
+      imu_suffix=""
+      parent_link="${parent_link}"
+      imu_topic="imu"
+      measurement_delay="0"
+      measurement_divisor="1"
+      mass_imu_sensor="0.00001"
+      gyroscope_noise_density="0.000175"
+      gyroscope_random_walk="0.0105"
+      gyroscope_bias_correlation_time="1000.0"
+      gyroscope_turn_on_bias_sigma= "0.09"
+      accelerometer_noise_density="0.003"
+      accelerometer_random_walk="0.18"
+      accelerometer_bias_correlation_time="300.0"
+      accelerometer_turn_on_bias_sigma="0.588">
       <inertia ixx="0.00001" ixy="0.0" ixz="0.0" iyy="0.00001" iyz="0.0" izz="0.00001" />
       <origin xyz="0 0 0" rpy="0 0 0" />

File: rotors_description/urdf/multirotor_base.xacro (robot description, xacro)
@@ -1,134 +1,155 @@
 <?xml version="1.0"?>
 <!--
-  Copyright 2015 Fadri Furrer, ASL, ETH Zurich, Switzerland
-  Copyright 2015 Michael Burri, ASL, ETH Zurich, Switzerland
-  Copyright 2015 Mina Kamel, ASL, ETH Zurich, Switzerland
-  Copyright 2015 Janosch Nikolic, ASL, ETH Zurich, Switzerland
-  Copyright 2015 Markus Achtelik, ASL, ETH Zurich, Switzerland
-  Licensed under the Apache License, Version 2.0 (the "License");
-  you may not use this file except in compliance with the License.
-  You may obtain a copy of the License at
-  http://www.apache.org/licenses/LICENSE-2.0
-  Unless required by applicable law or agreed to in writing, software
-  distributed under the License is distributed on an "AS IS" BASIS,
-  WITHOUT WARRANTIES OR CONDITIONS OF ANY KIND, either express or implied.
-  See the License for the specific language governing permissions and
-  limitations under the License.
+	Copyright 2015 Fadri Furrer, ASL, ETH Zurich, Switzerland
+	Copyright 2015 Michael Burri, ASL, ETH Zurich, Switzerland
+	Copyright 2015 Mina Kamel, ASL, ETH Zurich, Switzerland
+	Copyright 2015 Janosch Nikolic, ASL, ETH Zurich, Switzerland
+	Copyright 2015 Markus Achtelik, ASL, ETH Zurich, Switzerland
+	Licensed under the Apache License, Version 2.0 (the "License");
+	you may not use this file except in compliance with the License.
+	You may obtain a copy of the License at
+	http://www.apache.org/licenses/LICENSE-2.0
+	Unless required by applicable law or agreed to in writing, software
+	distributed under the License is distributed on an "AS IS" BASIS,
+	WITHOUT WARRANTIES OR CONDITIONS OF ANY KIND, either express or implied.
+	See the License for the specific language governing permissions and
+	limitations under the License.
 -->
 <robot xmlns:xacro="http://ros.org/wiki/xacro">
-  <!-- Macro for the inertia of a box -->
-  <xacro:macro name="box_inertia" params="x y z mass">
-    <inertia ixx="${0.0833333 * mass * (y*y + z*z)}" ixy="0.0" ixz="0.0"
-      iyy="${0.0833333 * mass * (x*x + z*z)}" iyz="0.0"
-      izz="${0.0833333 * mass * (x*x + y*y)}" />
-  </xacro:macro>
-  <!-- Macro for the inertial properties of a box -->
-  <xacro:macro name="box_inertial" params="x y z mass *origin">
-    <inertial>
-      <mass value="${mass}" />
-      <xacro:insert_block name="origin" />
-      <xacro:box_inertia x="${x}" y="${y}" z="${z}" mass="${mass}" />
-    </inertial>
-  </xacro:macro>
-  <!-- Main multirotor link -->
-  <xacro:macro name="multirotor_base_macro"
-    params="robot_namespace mass body_width body_height use_mesh_file mesh_file *inertia">
-    <link name="${robot_namespace}/base_link"></link>
-    <joint name="${robot_namespace}/base_joint" type="fixed">
-      <origin xyz="0 0 0" rpy="0 0 0" />
-      <parent link="${robot_namespace}/base_link" />
-      <child link="${robot_namespace}/base_link_inertia" />
-    </joint>
-    <link name="${robot_namespace}/base_link_inertia">
-      <inertial>
-        <mass value="${mass}" />  <!-- [kg] -->
-        <origin xyz="0 0 0" />
-        <xacro:insert_block name="inertia" />
-      </inertial>
-      <visual>
-        <origin xyz="0 0 0" rpy="0 0 0" />
-        <geometry>
-          <xacro:if value="${use_mesh_file}">
-            <mesh filename="${mesh_file}" scale="1 1 1" />
-          </xacro:if>
-          <xacro:unless value="${use_mesh_file}">
-            <box size="${body_width} ${body_width} ${body_height}"/> <!-- [m] [m] [m] -->
-          </xacro:unless>
-        </geometry>
-      </visual>
-      <collision>
-        <origin xyz="0 0 0" rpy="0 0 0" />
-        <geometry>
-          <box size="${body_width} ${body_width} ${body_height}" /> <!-- [m] [m] [m] -->
-        </geometry>
-      </collision>
-    </link>
-    <!-- attach multirotor_base_plugin to the base_link -->
-    <gazebo>
-      <plugin filename="librotors_gazebo_multirotor_base_plugin.so" name="multirotor_base_plugin">
-        <robotNamespace>${robot_namespace}</robotNamespace>
-        <linkName>${robot_namespace}/base_link</linkName>
-        <rotorVelocitySlowdownSim>${rotor_velocity_slowdown_sim}</rotorVelocitySlowdownSim>
-      </plugin>
-    </gazebo>
-  </xacro:macro>
-  <!-- Rotor joint and link -->
-  <xacro:macro name="vertical_rotor"
-    params="robot_namespace suffix direction motor_constant moment_constant parent mass_rotor radius_rotor time_constant_up time_constant_down max_rot_velocity motor_number rotor_drag_coefficient rolling_moment_coefficient color use_own_mesh mesh *origin *inertia">
-    <joint name="${robot_namespace}/rotor_${motor_number}_joint" type="continuous">
-      <xacro:insert_block name="origin" />
-      <axis xyz="0 0 1" />
-      <!-- TODO(ff): not currently set because it's not yet supported -->
-      <!-- <limit effort="2000" velocity="${max_rot_velocity}" /> -->
-      <parent link="${parent}" />
-      <child link="${robot_namespace}/rotor_${motor_number}" />
-    </joint>
-    <link name="${robot_namespace}/rotor_${motor_number}">
-      <inertial>
-        <mass value="${mass_rotor}" /> <!-- [kg] -->
-        <xacro:insert_block name="inertia" />
-      </inertial>
-      <visual>
-        <geometry>
-          <!-- <cylinder length="0.005" radius="${radius_rotor}"/> --> <!-- [m] -->
-          <xacro:if value="${use_own_mesh}">
-            <mesh filename="${mesh}"
-              scale="1 1 1" />
-          </xacro:if>
-          <xacro:unless value="${use_own_mesh}">
-            <mesh filename="package://rotors_description/meshes/propeller_${direction}.dae"
-              scale="${radius_rotor} ${radius_rotor} ${radius_rotor}" /> <!-- The propeller meshes have a radius of 1m -->
-            <!-- <box size="${2*radius_rotor} 0.01 0.005"/> -->
-          </xacro:unless>
-        </geometry>
-      </visual>
-      <collision>
-        <geometry>
-          <cylinder length="0.005" radius="${radius_rotor}" /> <!-- [m] -->
-        </geometry>
-      </collision>
-    </link>
-    <gazebo>
-      <plugin name="${robot_namespace}_${suffix}_motor_model" filename="librotors_gazebo_motor_model.so">
-        <robotNamespace>${robot_namespace}</robotNamespace>
-        <jointName>${robot_namespace}/rotor_${motor_number}_joint</jointName>
-        <linkName>${robot_namespace}/rotor_${motor_number}</linkName>
-        <turningDirection>${direction}</turningDirection>
-        <timeConstantUp>${time_constant_up}</timeConstantUp>
-        <timeConstantDown>${time_constant_down}</timeConstantDown>
-        <maxRotVelocity>${max_rot_velocity}</maxRotVelocity>
-        <motorConstant>${motor_constant}</motorConstant>
-        <momentConstant>${moment_constant}</momentConstant>
-        <commandSubTopic>gazebo/command/motor_speed</commandSubTopic>
-        <motorNumber>${motor_number}</motorNumber>
-        <rotorDragCoefficient>${rotor_drag_coefficient}</rotorDragCoefficient>
-        <rollingMomentCoefficient>${rolling_moment_coefficient}</rollingMomentCoefficient>
-        <motorSpeedPubTopic>motor_speed/${motor_number}</motorSpeedPubTopic>
-        <rotorVelocitySlowdownSim>${rotor_velocity_slowdown_sim}</rotorVelocitySlowdownSim>
-      </plugin>
-    </gazebo>
-    <gazebo reference="${robot_namespace}/rotor_${motor_number}">
-      <material>Gazebo/${color}</material>
-    </gazebo>
-  </xacro:macro>
+	<!-- Macro for the inertia of a box -->
+	<xacro:macro name="box_inertia" params="x y z mass">
+		<inertia ixx="${0.0833333 * mass * (y*y + z*z)}" ixy="0.0" ixz="0.0"
+			iyy="${0.0833333 * mass * (x*x + z*z)}" iyz="0.0"
+			izz="${0.0833333 * mass * (x*x + y*y)}" />
+	</xacro:macro>
+	<!-- Macro for the inertial properties of a box -->
+	<xacro:macro name="box_inertial" params="x y z mass *origin">
+		<inertial>
+			<mass value="${mass}" />
+			<xacro:insert_block name="origin" />
+			<xacro:box_inertia x="${x}" y="${y}" z="${z}" mass="${mass}" />
+		</inertial>
+	</xacro:macro>
+	<!-- Main multirotor link -->
+	<xacro:macro name="multirotor_base_macro"
+		params="robot_namespace mass body_width body_height use_mesh_file mesh_file *inertia">
+		<link name="${robot_namespace}/base_link"></link>
+		<joint name="${robot_namespace}/base_joint" type="fixed">
+			<origin xyz="0 0 0" rpy="0 0 0" />
+			<parent link="${robot_namespace}/base_link" />
+			<child link="${robot_namespace}/base_link_inertia" />
+		</joint>
+		<link name="${robot_namespace}/base_link_inertia">
+			<inertial>
+				<mass value="${mass}" />  <!-- [kg] -->
+				<origin xyz="0 0 0" />
+				<xacro:insert_block name="inertia" />
+			</inertial>
+			<visual>
+				<origin xyz="0 0 0" rpy="0 0 0" />
+				<geometry>
+					<xacro:if value="${use_mesh_file}">
+						<mesh filename="${mesh_file}" scale="1 1 1" />
+					</xacro:if>
+					<xacro:unless value="${use_mesh_file}">
+						<box size="${body_width} ${body_width} ${body_height}"/> <!-- [m] [m] [m] -->
+					</xacro:unless>
+				</geometry>
+			</visual>
+			<collision>
+				<origin xyz="0 0 0" rpy="0 0 0" />
+				<geometry>
+					<box size="${body_width} ${body_width} ${body_height}" /> <!-- [m] [m] [m] -->
+				</geometry>
+			</collision>
+		</link>
+		<!-- attach multirotor_base_plugin to the base_link -->
+		<gazebo>
+			<plugin filename="librotors_gazebo_multirotor_base_plugin.so" name="multirotor_base_plugin">
+				<robotNamespace>${robot_namespace}</robotNamespace>
+				<linkName>${robot_namespace}/base_link</linkName>
+				<rotorVelocitySlowdownSim>${rotor_velocity_slowdown_sim}</rotorVelocitySlowdownSim>
+			</plugin>
+		</gazebo>
+		<!-- <gazebo reference="${robot_namespace}/base_link">
+			<material>Gazebo/Black</material>
+		</gazebo> -->
+	</xacro:macro>
+	<!-- Rotor joint and link -->
+	<xacro:macro name="vertical_rotor"
+		params="robot_namespace suffix direction motor_constant moment_constant parent mass_rotor radius_rotor time_constant_up time_constant_down max_rot_velocity motor_number rotor_drag_coefficient rolling_moment_coefficient color use_own_mesh mesh *origin *inertia">
+		<joint name="${robot_namespace}/rotor_${motor_number}_joint" type="continuous">
+			<xacro:insert_block name="origin" />
+			<axis xyz="0 0 1" />
+			<!-- TODO(ff): not currently set because it's not yet supported -->
+			<!-- <limit effort="2000" velocity="${max_rot_velocity}" /> -->
+			<parent link="${parent}" />
+			<child link="${robot_namespace}/rotor_${motor_number}" />
+		</joint>
+		<link name="${robot_namespace}/rotor_${motor_number}">
+			<inertial>
+				<mass value="${mass_rotor}" /> <!-- [kg] -->
+				<xacro:insert_block name="inertia" />
+			</inertial>
+			<visual>
+				<geometry>
+					<!-- <cylinder length="0.005" radius="${radius_rotor}"/> --> <!-- [m] -->
+					<xacro:if value="${use_own_mesh}">
+						<mesh filename="${mesh}"
+							scale="1 1 1" />
+					</xacro:if>
+					<xacro:unless value="${use_own_mesh}">
+						<mesh filename="package://rotors_description/meshes/propeller_${direction}.dae"
+							scale="${radius_rotor} ${radius_rotor} ${radius_rotor}" /> <!-- The propeller meshes have a radius of 1m -->
+						<!-- <box size="${2*radius_rotor} 0.01 0.005"/> -->
+					</xacro:unless>
+				</geometry>
+			</visual>
+			<collision>
+				<geometry>
+					<cylinder length="0.005" radius="${radius_rotor}" /> <!-- [m] -->
+				</geometry>
+			</collision>
+		</link>
+		<gazebo>
+			<plugin name="${robot_namespace}_${suffix}_motor_model" filename="librotors_gazebo_motor_model.so">
+				<robotNamespace>${robot_namespace}</robotNamespace>
+				<jointName>${robot_namespace}/rotor_${motor_number}_joint</jointName>
+				<linkName>${robot_namespace}/rotor_${motor_number}</linkName>
+				<turningDirection>${direction}</turningDirection>
+				<timeConstantUp>${time_constant_up}</timeConstantUp>
+				<timeConstantDown>${time_constant_down}</timeConstantDown>
+				<maxRotVelocity>${max_rot_velocity}</maxRotVelocity>
+				<motorConstant>${motor_constant}</motorConstant>
+				<momentConstant>${moment_constant}</momentConstant>
+				<commandSubTopic>gazebo/command/motor_speed</commandSubTopic>
+				<motorNumber>${motor_number}</motorNumber>
+				<rotorDragCoefficient>${rotor_drag_coefficient}</rotorDragCoefficient>
+				<rollingMomentCoefficient>${rolling_moment_coefficient}</rollingMomentCoefficient>
+				<motorSpeedPubTopic>motor_speed/${motor_number}</motorSpeedPubTopic>
+				<rotorVelocitySlowdownSim>${rotor_velocity_slowdown_sim}</rotorVelocitySlowdownSim>
+			</plugin>
+		</gazebo>
+		<gazebo reference="${robot_namespace}/rotor_${motor_number}">
+			<material>Gazebo/${color}</material>
+		</gazebo>
+	</xacro:macro>
+	<xacro:macro name="vertical_motor"
+		params="robot_namespace suffix parent radius_rotor motor_number *origin">
+		<!-- Motor visual -->
+		<joint name="${robot_namespace}/motor_${motor_number}_joint" type="fixed">
+			<xacro:insert_block name="origin" />
+			<!-- <axis xyz="0 0 1" /> -->
+			<parent link="${parent}" />
+			<child link="${robot_namespace}/motor_${motor_number}" />
+		</joint>
+		<link name="${robot_namespace}/motor_${motor_number}">
+			<visual>
+				<geometry>
+					<mesh filename="package://rotors_description/meshes/edrone_motor.stl"
+						scale="0.001 0.001 0.001" />
+				</geometry>
+			</visual>
+		</link>
+	</xacro:macro>
 </robot>
