Commit message: Tuned ardrone as well

File: rotors_description/urdf/ardrone_base.xacro (robot description, xacro)
@@ -4,4 +4,5 @@
   <!-- Instantiate ardrone "mechanics" -->
   <xacro:include filename="$(find rotors_description)/urdf/ardrone.xacro" />
+    <xacro:include filename="$(find rotors_description)/urdf/whycon_marker_file.xacro"/>
   <!-- Instantiate a controller. -->
   <xacro:controller_plugin_macro namespace="${namespace}" imu_sub_topic="imu" />
@@ -23,3 +24,4 @@
       wait_to_record_bag="$(arg wait_to_record_bag)" />
   </xacro:if>
+  <xacro:whycon_marker namespace="${namespace}" marker="whycon_marker" marker_width="0.001" marker_radius="0.01"/>
 </robot>

File: rotors_description/urdf/edrone.xacro (robot description, xacro)
@@ -6,5 +6,5 @@
   <!-- Properties (Taken from Novel Dynamic Inversion Architecture Design for Quadrocopter Control by Jian Wang et al.) -->
   <xacro:property name="namespace" value="$(arg mav_name)" />
-  <xacro:property name="rotor_velocity_slowdown_sim" value="5" />
+  <xacro:property name="rotor_velocity_slowdown_sim" value="10" />
   <xacro:property name="use_mesh_file" value="true" />
   <!-- <xacro:property name="mesh_file" value="package://rotors_description/meshes/crazyflie2.dae" /> -->

File: rotors_description/urdf/whycon_marker_file.xacro (robot description, xacro)
@@ -21,5 +21,7 @@
 		<joint name="${marker}_joint" type="fixed">
 			<!-- <origin xyz="0 0 0.095" rpy="0 0 0"/> -->
-			<origin xyz="0 0 0.015" rpy="0 0 0"/>
+			<!-- <origin xyz="0 0 0.015" rpy="0 0 0"/> -->
+			<origin xyz="0 0 0.03" rpy="0 0 0"/>
+			<!-- ^^ for ardrone -->
 			<parent link="${namespace}/base_link"/>
 			<child link="${marker}_link"/>
