Commit message: Changed edrone motor directions

File: rotors_description/urdf/edrone.xacro (robot description, xacro)
@@ -54,5 +54,5 @@
     robot_namespace="${namespace}"
     suffix="front_right"
-    direction="ccw"
+    direction="cw"
     motor_constant="${motor_constant}"
     moment_constant="${moment_constant}"
@@ -69,5 +69,5 @@
     use_own_mesh="false"
     mesh="">
-    <origin xyz="${sqrt2by2 * arm_length} -${sqrt2by2 * arm_length} ${rotor_offset_top}" rpy="0 0 0" />
+    <origin xyz="${sqrt2by2 * arm_length} ${sqrt2by2 * arm_length} ${rotor_offset_top}" rpy="0 0 0" />
     <xacro:insert_block name="rotor_inertia" />
   </xacro:vertical_rotor>
@@ -78,9 +78,9 @@
     robot_namespace="${namespace}"
     suffix="front_right">
-    <origin xyz="${sqrt2by2 * arm_length} -${sqrt2by2 * arm_length} ${motor_offset_top}" rpy="1.570796327 0 0"/>
+    <origin xyz="${sqrt2by2 * arm_length} ${sqrt2by2 * arm_length} ${motor_offset_top}" rpy="1.570796327 0 0"/>
   </xacro:vertical_motor>
   <xacro:vertical_rotor
     robot_namespace="${namespace}"
-    suffix="back_left"
+    suffix="front_left"
     direction="ccw"
     motor_constant="${motor_constant}"
@@ -110,5 +110,5 @@
   </xacro:vertical_motor>
   <xacro:vertical_rotor robot_namespace="${namespace}"
-    suffix="front_left"
+    suffix="back_left"
     direction="cw"
     motor_constant="${motor_constant}"
@@ -126,5 +126,5 @@
     use_own_mesh="false"
     mesh="">
-    <origin xyz="${sqrt2by2 * arm_length} ${sqrt2by2 * arm_length} ${rotor_offset_top}" rpy="0 0 0" />
+    <origin xyz="-${sqrt2by2 * arm_length} -${sqrt2by2 * arm_length} ${rotor_offset_top}" rpy="0 0 0" />
     <xacro:insert_block name="rotor_inertia" />
   </xacro:vertical_rotor>
@@ -135,9 +135,9 @@
     robot_namespace="${namespace}"
     suffix="front_left">
-    <origin xyz="${sqrt2by2 * arm_length} ${sqrt2by2 * arm_length} ${motor_offset_top}" rpy="1.570796327 0 0"/>
+    <origin xyz="-${sqrt2by2 * arm_length} -${sqrt2by2 * arm_length} ${motor_offset_top}" rpy="1.570796327 0 0"/>
   </xacro:vertical_motor>
   <xacro:vertical_rotor robot_namespace="${namespace}"
     suffix="back_right"
-    direction="cw"
+    direction="ccw"
     motor_constant="${motor_constant}"
     moment_constant="${moment_constant}"
@@ -154,5 +154,5 @@
     use_own_mesh="false"
     mesh="">
-    <origin xyz="-${sqrt2by2 * arm_length} -${sqrt2by2 * arm_length} ${rotor_offset_top}" rpy="0 0 0" />
+    <origin xyz="${sqrt2by2 * arm_length} -${sqrt2by2 * arm_length} ${rotor_offset_top}" rpy="0 0 0" />
     <xacro:insert_block name="rotor_inertia" />
   </xacro:vertical_rotor>
@@ -163,5 +163,5 @@
     robot_namespace="${namespace}"
     suffix="back_right">
-    <origin xyz="-${sqrt2by2 * arm_length } -${sqrt2by2 * arm_length} ${motor_offset_top}" rpy="1.570796327 0 0"/>
+    <origin xyz="${sqrt2by2 * arm_length } -${sqrt2by2 * arm_length} ${motor_offset_top}" rpy="1.570796327 0 0"/>
   </xacro:vertical_motor>
 </robot>

File: rotors_description/urdf/whycon_marker_file.xacro (robot description, xacro)
@@ -21,6 +21,6 @@
 		<joint name="${marker}_joint" type="fixed">
 			<!-- <origin xyz="0 0 0.095" rpy="0 0 0"/> -->
-			<!-- <origin xyz="0 0 0.015" rpy="0 0 0"/> -->
-			<origin xyz="0 0 0.03" rpy="0 0 0"/>
+			<origin xyz="0 0 0.015" rpy="0 0 0"/>
+			<!-- <origin xyz="0 0 0.03" rpy="0 0 0"/> -->
 			<!-- ^^ for ardrone -->
 			<parent link="${namespace}/base_link"/>

Commit message: Changed edrone motors back

File: rotors_description/urdf/edrone.xacro (robot description, xacro)
@@ -54,5 +54,5 @@
     robot_namespace="${namespace}"
     suffix="front_right"
-    direction="cw"
+    direction="ccw"
     motor_constant="${motor_constant}"
     moment_constant="${moment_constant}"
@@ -69,5 +69,5 @@
     use_own_mesh="false"
     mesh="">
-    <origin xyz="${sqrt2by2 * arm_length} ${sqrt2by2 * arm_length} ${rotor_offset_top}" rpy="0 0 0" />
+    <origin xyz="${sqrt2by2 * arm_length} -${sqrt2by2 * arm_length} ${rotor_offset_top}" rpy="0 0 0" />
     <xacro:insert_block name="rotor_inertia" />
   </xacro:vertical_rotor>
@@ -78,9 +78,9 @@
     robot_namespace="${namespace}"
     suffix="front_right">
-    <origin xyz="${sqrt2by2 * arm_length} ${sqrt2by2 * arm_length} ${motor_offset_top}" rpy="1.570796327 0 0"/>
+    <origin xyz="${sqrt2by2 * arm_length} -${sqrt2by2 * arm_length} ${motor_offset_top}" rpy="1.570796327 0 0"/>
   </xacro:vertical_motor>
   <xacro:vertical_rotor
     robot_namespace="${namespace}"
-    suffix="front_left"
+    suffix="back_left"
     direction="ccw"
     motor_constant="${motor_constant}"
@@ -110,5 +110,5 @@
   </xacro:vertical_motor>
   <xacro:vertical_rotor robot_namespace="${namespace}"
-    suffix="back_left"
+    suffix="front_left"
     direction="cw"
     motor_constant="${motor_constant}"
@@ -126,5 +126,5 @@
     use_own_mesh="false"
     mesh="">
-    <origin xyz="-${sqrt2by2 * arm_length} -${sqrt2by2 * arm_length} ${rotor_offset_top}" rpy="0 0 0" />
+    <origin xyz="${sqrt2by2 * arm_length} ${sqrt2by2 * arm_length} ${rotor_offset_top}" rpy="0 0 0" />
     <xacro:insert_block name="rotor_inertia" />
   </xacro:vertical_rotor>
@@ -135,9 +135,9 @@
     robot_namespace="${namespace}"
     suffix="front_left">
-    <origin xyz="-${sqrt2by2 * arm_length} -${sqrt2by2 * arm_length} ${motor_offset_top}" rpy="1.570796327 0 0"/>
+    <origin xyz="${sqrt2by2 * arm_length} ${sqrt2by2 * arm_length} ${motor_offset_top}" rpy="1.570796327 0 0"/>
   </xacro:vertical_motor>
   <xacro:vertical_rotor robot_namespace="${namespace}"
     suffix="back_right"
-    direction="ccw"
+    direction="cw"
     motor_constant="${motor_constant}"
     moment_constant="${moment_constant}"
@@ -154,5 +154,5 @@
     use_own_mesh="false"
     mesh="">
-    <origin xyz="${sqrt2by2 * arm_length} -${sqrt2by2 * arm_length} ${rotor_offset_top}" rpy="0 0 0" />
+    <origin xyz="-${sqrt2by2 * arm_length} -${sqrt2by2 * arm_length} ${rotor_offset_top}" rpy="0 0 0" />
     <xacro:insert_block name="rotor_inertia" />
   </xacro:vertical_rotor>
@@ -163,5 +163,5 @@
     robot_namespace="${namespace}"
     suffix="back_right">
-    <origin xyz="${sqrt2by2 * arm_length } -${sqrt2by2 * arm_length} ${motor_offset_top}" rpy="1.570796327 0 0"/>
+    <origin xyz="-${sqrt2by2 * arm_length } -${sqrt2by2 * arm_length} ${motor_offset_top}" rpy="1.570796327 0 0"/>
   </xacro:vertical_motor>
 </robot>
