Commit message: edrone_big added

File: rotors_description/urdf/multirotor_base.xacro (robot description, xacro)
@@ -22,54 +22,54 @@
 			iyy="${0.0833333 * mass * (x*x + z*z)}" iyz="0.0"
 			izz="${0.0833333 * mass * (x*x + y*y)}" />
-	</xacro:macro>
-	<!-- Macro for the inertial properties of a box -->
-	<xacro:macro name="box_inertial" params="x y z mass *origin">
-		<inertial>
-			<mass value="${mass}" />
-			<xacro:insert_block name="origin" />
-			<xacro:box_inertia x="${x}" y="${y}" z="${z}" mass="${mass}" />
-		</inertial>
-	</xacro:macro>
-	<!-- Main multirotor link -->
-	<xacro:macro name="multirotor_base_macro"
-		params="robot_namespace mass body_width body_height use_mesh_file mesh_file *inertia">
-		<link name="${robot_namespace}/base_link"></link>
-		<joint name="${robot_namespace}/base_joint" type="fixed">
-			<origin xyz="0 0 0" rpy="0 0 0" />
-			<parent link="${robot_namespace}/base_link" />
-			<child link="${robot_namespace}/base_link_inertia" />
-		</joint>
-		<link name="${robot_namespace}/base_link_inertia">
+		</xacro:macro>
+		<!-- Macro for the inertial properties of a box -->
+		<xacro:macro name="box_inertial" params="x y z mass *origin">
 			<inertial>
-				<mass value="${mass}" />  <!-- [kg] -->
-				<origin xyz="0 0 0" />
-				<xacro:insert_block name="inertia" />
+				<mass value="${mass}" />
+				<xacro:insert_block name="origin" />
+				<xacro:box_inertia x="${x}" y="${y}" z="${z}" mass="${mass}" />
 			</inertial>
-			<visual>
+		</xacro:macro>
+		<!-- Main multirotor link -->
+		<xacro:macro name="multirotor_base_macro"
+			params="robot_namespace mass body_width body_height use_mesh_file mesh_file *inertia">
+			<link name="${robot_namespace}/base_link"></link>
+			<joint name="${robot_namespace}/base_joint" type="fixed">
 				<origin xyz="0 0 0" rpy="0 0 0" />
-				<geometry>
-					<xacro:if value="${use_mesh_file}">
-						<mesh filename="${mesh_file}" scale="1 1 1" />
-					</xacro:if>
-					<xacro:unless value="${use_mesh_file}">
-						<box size="${body_width} ${body_width} ${body_height}"/> <!-- [m] [m] [m] -->
-					</xacro:unless>
-				</geometry>
-			</visual>
-			<collision>
-				<origin xyz="0 0 0" rpy="0 0 0" />
-				<geometry>
-					<box size="${body_width} ${body_width} ${body_height}" /> <!-- [m] [m] [m] -->
-				</geometry>
-			</collision>
-		</link>
-		<!-- attach multirotor_base_plugin to the base_link -->
-		<gazebo>
-			<plugin filename="librotors_gazebo_multirotor_base_plugin.so" name="multirotor_base_plugin">
-				<robotNamespace>${robot_namespace}</robotNamespace>
-				<linkName>${robot_namespace}/base_link</linkName>
-				<rotorVelocitySlowdownSim>${rotor_velocity_slowdown_sim}</rotorVelocitySlowdownSim>
-			</plugin>
-		</gazebo>
+				<parent link="${robot_namespace}/base_link" />
+				<child link="${robot_namespace}/base_link_inertia" />
+			</joint>
+			<link name="${robot_namespace}/base_link_inertia">
+				<inertial>
+					<mass value="${mass}" />  <!-- [kg] -->
+					<origin xyz="0 0 0" />
+					<xacro:insert_block name="inertia" />
+				</inertial>
+				<visual>
+					<origin xyz="0 0 0" rpy="0 0 0" />
+					<geometry>
+						<xacro:if value="${use_mesh_file}">
+							<mesh filename="${mesh_file}" scale="1 1 1" />
+						</xacro:if>
+						<xacro:unless value="${use_mesh_file}">
+							<box size="${body_width} ${body_width} ${body_height}"/> <!-- [m] [m] [m] -->
+						</xacro:unless>
+					</geometry>
+				</visual>
+				<collision>
+					<origin xyz="0 0 0" rpy="0 0 0" />
+					<geometry>
+						<box size="${body_width} ${body_width} ${body_height}" /> <!-- [m] [m] [m] -->
+					</geometry>
+				</collision>
+			</link>
+			<!-- attach multirotor_base_plugin to the base_link -->
+			<gazebo>
+				<plugin filename="librotors_gazebo_multirotor_base_plugin.so" name="multirotor_base_plugin">
+					<robotNamespace>${robot_namespace}</robotNamespace>
+					<linkName>${robot_namespace}/base_link</linkName>
+					<rotorVelocitySlowdownSim>${rotor_velocity_slowdown_sim}</rotorVelocitySlowdownSim>
+				</plugin>
+			</gazebo>
 		<!-- <gazebo reference="${robot_namespace}/base_link">
 			<material>Gazebo/Black</material>
@@ -98,58 +98,60 @@
 						<mesh filename="${mesh}"
 							scale="1 1 1" />
-					</xacro:if>
-					<xacro:unless value="${use_own_mesh}">
-						<mesh filename="package://rotors_description/meshes/propeller_${direction}.dae"
-							scale="${radius_rotor} ${radius_rotor} ${radius_rotor}" /> <!-- The propeller meshes have a radius of 1m -->
-						<!-- <box size="${2*radius_rotor} 0.01 0.005"/> -->
-					</xacro:unless>
-				</geometry>
-			</visual>
-			<collision>
-				<geometry>
-					<cylinder length="0.005" radius="${radius_rotor}" /> <!-- [m] -->
-				</geometry>
-			</collision>
-		</link>
-		<gazebo>
-			<plugin name="${robot_namespace}_${suffix}_motor_model" filename="librotors_gazebo_motor_model.so">
-				<robotNamespace>${robot_namespace}</robotNamespace>
-				<jointName>${robot_namespace}/rotor_${motor_number}_joint</jointName>
-				<linkName>${robot_namespace}/rotor_${motor_number}</linkName>
-				<turningDirection>${direction}</turningDirection>
-				<timeConstantUp>${time_constant_up}</timeConstantUp>
-				<timeConstantDown>${time_constant_down}</timeConstantDown>
-				<maxRotVelocity>${max_rot_velocity}</maxRotVelocity>
-				<motorConstant>${motor_constant}</motorConstant>
-				<momentConstant>${moment_constant}</momentConstant>
-				<commandSubTopic>gazebo/command/motor_speed</commandSubTopic>
-				<motorNumber>${motor_number}</motorNumber>
-				<rotorDragCoefficient>${rotor_drag_coefficient}</rotorDragCoefficient>
-				<rollingMomentCoefficient>${rolling_moment_coefficient}</rollingMomentCoefficient>
-				<motorSpeedPubTopic>motor_speed/${motor_number}</motorSpeedPubTopic>
-				<rotorVelocitySlowdownSim>${rotor_velocity_slowdown_sim}</rotorVelocitySlowdownSim>
-			</plugin>
-		</gazebo>
-		<gazebo reference="${robot_namespace}/rotor_${motor_number}">
-			<material>Gazebo/${color}</material>
-		</gazebo>
-	</xacro:macro>
-	<xacro:macro name="vertical_motor"
-		params="robot_namespace suffix parent radius_rotor motor_number *origin">
-		<!-- Motor visual -->
-		<joint name="${robot_namespace}/motor_${motor_number}_joint" type="fixed">
-			<xacro:insert_block name="origin" />
-			<!-- <axis xyz="0 0 1" /> -->
-			<parent link="${parent}" />
-			<child link="${robot_namespace}/motor_${motor_number}" />
-		</joint>
-		<link name="${robot_namespace}/motor_${motor_number}">
-			<visual>
-				<geometry>
+						</xacro:if>
+						<xacro:unless value="${use_own_mesh}">
+							<mesh filename="package://rotors_description/meshes/propeller_${direction}.dae"
+								scale="${radius_rotor} ${radius_rotor} ${radius_rotor}" /> <!-- The propeller meshes have a radius of 1m -->
+								<!-- <box size="${2*radius_rotor} 0.01 0.005"/> -->
+							</xacro:unless>
+						</geometry>
+					</visual>
+					<collision>
+						<geometry>
+							<cylinder length="0.005" radius="${radius_rotor}" /> <!-- [m] -->
+						</geometry>
+					</collision>
+				</link>
+				<gazebo>
+					<plugin name="${robot_namespace}_${suffix}_motor_model" filename="librotors_gazebo_motor_model.so">
+						<robotNamespace>${robot_namespace}</robotNamespace>
+						<jointName>${robot_namespace}/rotor_${motor_number}_joint</jointName>
+						<linkName>${robot_namespace}/rotor_${motor_number}</linkName>
+						<turningDirection>${direction}</turningDirection>
+						<timeConstantUp>${time_constant_up}</timeConstantUp>
+						<timeConstantDown>${time_constant_down}</timeConstantDown>
+						<maxRotVelocity>${max_rot_velocity}</maxRotVelocity>
+						<motorConstant>${motor_constant}</motorConstant>
+						<momentConstant>${moment_constant}</momentConstant>
+						<commandSubTopic>gazebo/command/motor_speed</commandSubTopic>
+						<motorNumber>${motor_number}</motorNumber>
+						<rotorDragCoefficient>${rotor_drag_coefficient}</rotorDragCoefficient>
+						<rollingMomentCoefficient>${rolling_moment_coefficient}</rollingMomentCoefficient>
+						<motorSpeedPubTopic>motor_speed/${motor_number}</motorSpeedPubTopic>
+						<rotorVelocitySlowdownSim>${rotor_velocity_slowdown_sim}</rotorVelocitySlowdownSim>
+					</plugin>
+				</gazebo>
+				<gazebo reference="${robot_namespace}/rotor_${motor_number}">
+					<material>Gazebo/${color}</material>
+				</gazebo>
+			</xacro:macro>
+			<xacro:macro name="vertical_motor"
+				params="robot_namespace suffix parent radius_rotor motor_number *origin">
+				<!-- Motor visual -->
+				<joint name="${robot_namespace}/motor_${motor_number}_joint" type="fixed">
+					<xacro:insert_block name="origin" />
+					<!-- <axis xyz="0 0 1" /> -->
+					<parent link="${parent}" />
+					<child link="${robot_namespace}/motor_${motor_number}" />
+				</joint>
+				<link name="${robot_namespace}/motor_${motor_number}">
+					<visual>
+						<geometry>
 					<mesh filename="package://rotors_description/meshes/edrone_motor.stl"
-						scale="0.001 0.001 0.001" />
-				</geometry>
-			</visual>
-		</link>
-	</xacro:macro>
+scale="0.002769 0.002769 0.002769" />
+<!-- 											<mesh filename="package://rotors_description/meshes/edrone_motor.stl"
+scale="0.001 0.001 0.001" /> -->
+</geometry>
+</visual>
+</link>
+</xacro:macro>
 </robot>

File: rotors_description/urdf/whycon_marker_file.xacro (robot description, xacro)
@@ -21,6 +21,6 @@
 		<joint name="${marker}_joint" type="fixed">
 			<!-- <origin xyz="0 0 0.095" rpy="0 0 0"/> -->
-			<origin xyz="0 0 0.015" rpy="0 0 0"/>
-			<!-- <origin xyz="0 0 0.03" rpy="0 0 0"/> -->
+			<!-- <origin xyz="0 0 0.015" rpy="0 0 0"/> -->
+			<origin xyz="0 0 0.035" rpy="0 0 0"/>
 			<!-- ^^ for ardrone -->
 			<parent link="${namespace}/base_link"/>
@@ -37,34 +37,9 @@
 					<origin xyz="-0.01838 0 0" rpy="0 1.570796327 0"/>
 					<geometry>
-						<!-- <cylinder length="${marker_width}" radius="${marker_radius}"/> -->
-						<!-- <box size="${marker_radius} ${marker_radius} ${marker_width}"/> -->
-						<!-- <mesh filename="model://marker0/meshes/Marker0.dae" scale="0.25 0.075 0.075" /> -->
-						<!-- <mesh filename="package://rotors_description/models/marker0/meshes/Marker1.dae" scale="0.25 0.075 0.075"/> -->
+						<!-- <mesh filename="package://rotors_gazebo/models/marker0/meshes/Marker1.dae" scale="0.25 0.075 0.075"/> -->
 						<mesh filename="package://rotors_gazebo/models/marker0/meshes/Marker1.dae" scale="0.25 0.075 0.075"/>
-						<!-- <uri>model://marker0/meshes/Marker0.dae</uri> -->
 					</geometry>
-					<!-- <material name="WhyconMarkerTexture"/> -->
-					<!-- <material>
-						<texture filename="package://rotors_description/models/Marker0/meshes/Marker0.dae"/>
-					</material> -->
-					<!-- <material name="Marker1_png"> -->
-					<!-- <script> -->
-					<!-- <uri>models://marker0/materials/scripts/whycon_marker.material</uri> -->
-					<!-- <name>Gazebo/WhyconMarkerTexture</name> -->
-					<!-- <texture filename="package://rotors_description/models/marker0/meshes/Marker0.dae" /> -->
-					<!-- </script> -->
-					<!-- </material> -->
 				</visual>
-				<collision>
-					<geometry>
-						<!-- <cylinder length="${marker_width}" radius="${marker_radius}"/> -->
-						<box size="${marker_radius} ${marker_radius} ${marker_width}"/>
-					</geometry>
-				</collision>
 			</link>
-			<!-- <gazebo reference="${marker}_link"> -->
-				<!-- <material>Gazebo/Marker1_png</material> -->
-				<!-- <material>Gazebo/WhyconMarkerTexture</material>
-			</gazebo> -->
 		</xacro:macro>
 	</robot>
