Commit message: edrone_big's whycon marker fixed

File: rotors_description/urdf/whycon_marker_file.xacro (robot description, xacro)
@@ -1,26 +1,11 @@
 <?xml version="1.0"?>
 <robot name="crazyflie2" xmlns:xacro="http://ros.org/wiki/xacro">
-	<material name="Black">
-		<color rgba="0.0 0.0 0.0 1.0"/>
-	</material>
-	<material name="Red">
-		<color rgba="0.8 0.0 0.0 1.0"/>
-	</material>
-	<material name="Green">
-		<color rgba="0.0 0.8 0.0 1.0"/>
-	</material>
-	<material name="White">
-		<color rgba="1.0 1.0 1.0 1.0"/>
-	</material>
-	<material name="Blue">
-		<color rgba="0.0 0.0 0.8 1.0"/>
-	</material>
-	--&gt;
-	<!-- <xacro:include filename="$(find rotors_description)/urdf/materials.urdf.xacro"/> -->
 	<xacro:macro name="whycon_marker" params="namespace marker_width marker_radius marker">
 		<joint name="${marker}_joint" type="fixed">
 			<!-- <origin xyz="0 0 0.095" rpy="0 0 0"/> -->
+			<!-- edrone's positioning -->
 			<!-- <origin xyz="0 0 0.015" rpy="0 0 0"/> -->
-			<origin xyz="0 0 0.035" rpy="0 0 0"/>
+			<!-- edrone_big's positioning -->
+			<origin xyz="0 0 0.04" rpy="0 0 0"/>
 			<!-- ^^ for ardrone -->
 			<parent link="${namespace}/base_link"/>
@@ -35,8 +20,13 @@
 				</inertial> -->
 				<visual name='Marker0'>
-					<origin xyz="-0.01838 0 0" rpy="0 1.570796327 0"/>
+					<!-- edrone's positioning -->
+					<!-- <origin xyz="-0.01838 0 0" rpy="0 1.570796327 0"/> -->
+					<!-- edrone_big's positioning -->
+					<origin xyz="-0.05875 0 0" rpy="0 1.570796327 0"/>
 					<geometry>
+						<!-- edrone's scalling factors -->
 						<!-- <mesh filename="package://rotors_gazebo/models/marker0/meshes/Marker1.dae" scale="0.25 0.075 0.075"/> -->
-						<mesh filename="package://rotors_gazebo/models/marker0/meshes/Marker1.dae" scale="0.25 0.075 0.075"/>
+						<!-- edrone_big's scalling factors -->
+						<mesh filename="package://rotors_gazebo/models/marker0/meshes/Marker1.dae" scale="0.5 0.2375 0.2375"/>
 					</geometry>
 				</visual>
