Commit message: added crazyflie2, fixed collision

File: rotors_description/urdf/crazyflie2.xacro (robot description, xacro)
@@ -1,26 +1,33 @@
 <?xml version="1.0"?>
 <!--
-  TO BE CHANGED TO EDRONE.xacro due to changes in arm length and extra motors
+  Copyright 2018 Giuseppe Silano, University of Sannio in Benevento, Italy
+  Copyright 2018 Emanuele Aucone, University of Sannio in Benevento, Italy
+  Copyright 2018 Benjamin Rodriguez, MIT, USA
+  Copyright 2018 Luigi Iannelli, University of Sannio in Benevento, Italy
+  Licensed under the Apache License, Version 2.0 (the "License");
+  you may not use this file except in compliance with the License.
+  You may obtain a copy of the License at
+  http://www.apache.org/licenses/LICENSE-2.0
+  Unless required by applicable law or agreed to in writing, software
+  distributed under the License is distributed on an "AS IS" BASIS,
+  WITHOUT WARRANTIES OR CONDITIONS OF ANY KIND, either express or implied.
+  See the License for the specific language governing permissions and
+  limitations under the License.
 -->
-<robot name="edrone" xmlns:xacro="http://ros.org/wiki/xacro">
+<robot name="crazyflie2" xmlns:xacro="http://ros.org/wiki/xacro">
   <!-- Properties (Taken from Novel Dynamic Inversion Architecture Design for Quadrocopter Control by Jian Wang et al.) -->
   <xacro:property name="namespace" value="$(arg mav_name)" />
-  <xacro:property name="rotor_velocity_slowdown_sim" value="5" />
+  <xacro:property name="rotor_velocity_slowdown_sim" value="50" />
   <xacro:property name="use_mesh_file" value="true" />
-  <!-- <xacro:property name="mesh_file" value="package://rotors_description/meshes/crazyflie2.dae" /> -->
-  <xacro:property name="mesh_file" value="package://rotors_description/meshes/edrone_frame.stl" />
-  <xacro:property name="mass" value="0.027" /> <!-- [kg] -->
-  <xacro:property name="body_width" value="0.11" /> <!-- [m] -->
-  <xacro:property name="body_height" value="0.036" /> <!-- [m] -->
-  <xacro:property name="mass_rotor" value="0.00033" /> <!-- [kg] -->
-  <xacro:property name="arm_length" value="0.065" /> <!-- [m] -->
-  <!-- <xacro:property name="rotor_offset_top" value="0.024" /> --> <!-- [m] -->
-  <xacro:property name="rotor_offset_top" value="0.015" />
-  <xacro:property name="motor_offset_top" value="-0.015" />
+  <xacro:property name="mesh_file" value="package://rotors_description/meshes/crazyflie2.dae" />
+  <xacro:property name="mass" value="0.025" /> <!-- [kg] -->
+  <xacro:property name="body_width" value="0.045" /> <!-- [m] -->
+  <xacro:property name="body_height" value="0.03" /> <!-- [m] -->
+  <xacro:property name="mass_rotor" value="0.0005" /> <!-- [kg] -->
+  <xacro:property name="arm_length" value="0.046" /> <!-- [m] -->
+  <xacro:property name="rotor_offset_top" value="0.024" /> <!-- [m] -->
   <xacro:property name="radius_rotor" value="0.0225" /> <!-- [m] -->
   <!-- Forster's -->
-  <!-- [kg m/s^2] -->
-  <xacro:property name="motor_constant" value="1.28192e-08" />
-  <!-- <xacro:property name="motor_constant" value="1e-07" />  -->
+  <xacro:property name="motor_constant" value="1.28192e-08" /> <!-- [kg m/s^2] -->
   <xacro:property name="moment_constant" value="5.964552e-03" /> <!-- [m] -->
   <xacro:property name="time_constant_up" value="0.0125" /> <!-- [s] -->
@@ -32,9 +39,9 @@
   <!-- Property Blocks -->
   <xacro:property name="body_inertia">
-    <inertia ixx="1.657171e-06" ixy="0.0" ixz="0.0" iyy="1.657171e-06" iyz="0.0" izz="2.9261652e-06" />
+    <inertia ixx="1.657171e-05" ixy="0.0" ixz="0.0" iyy="1.657171e-05" iyz="0.0" izz="2.9261652e-05" />
   </xacro:property>
   <!-- inertia of a single rotor, assuming it is a cuboid. Height=0.4mm, width=0.8mm -->
   <xacro:property name="rotor_inertia">
-    <xacro:box_inertia x="${radius_rotor}" y="0.001" z="0.0003" mass="${mass_rotor*rotor_velocity_slowdown_sim}" />
+    <xacro:box_inertia x="${radius_rotor}" y="0.007" z="0.003" mass="${mass_rotor*rotor_velocity_slowdown_sim}" />
   </xacro:property>
   <!-- Included URDF Files -->
@@ -72,12 +79,4 @@
     <xacro:insert_block name="rotor_inertia" />
   </xacro:vertical_rotor>
-  <xacro:vertical_motor
-    radius_rotor="${radius_rotor}"
-    motor_number="0"
-    parent="${namespace}/base_link"
-    robot_namespace="${namespace}"
-    suffix="front_right">
-    <origin xyz="${sqrt2by2 * arm_length} -${sqrt2by2 * arm_length} ${motor_offset_top}" rpy="1.570796327 0 0"/>
-  </xacro:vertical_motor>
   <xacro:vertical_rotor
     robot_namespace="${namespace}"
@@ -101,12 +100,4 @@
     <xacro:insert_block name="rotor_inertia" />
   </xacro:vertical_rotor>
-  <xacro:vertical_motor
-    radius_rotor="${radius_rotor}"
-    motor_number="1"
-    parent="${namespace}/base_link"
-    robot_namespace="${namespace}"
-    suffix="back_left">
-    <origin xyz="-${sqrt2by2 * arm_length} ${sqrt2by2 * arm_length} ${motor_offset_top}" rpy="1.570796327 0 0"/>
-  </xacro:vertical_motor>
   <xacro:vertical_rotor robot_namespace="${namespace}"
     suffix="front_left"
@@ -129,12 +120,4 @@
     <xacro:insert_block name="rotor_inertia" />
   </xacro:vertical_rotor>
-  <xacro:vertical_motor
-    radius_rotor="${radius_rotor}"
-    motor_number="2"
-    parent="${namespace}/base_link"
-    robot_namespace="${namespace}"
-    suffix="front_left">
-    <origin xyz="${sqrt2by2 * arm_length} ${sqrt2by2 * arm_length} ${motor_offset_top}" rpy="1.570796327 0 0"/>
-  </xacro:vertical_motor>
   <xacro:vertical_rotor robot_namespace="${namespace}"
     suffix="back_right"
@@ -157,11 +140,3 @@
     <xacro:insert_block name="rotor_inertia" />
   </xacro:vertical_rotor>
-  <xacro:vertical_motor
-    radius_rotor="${radius_rotor}"
-    motor_number="3"
-    parent="${namespace}/base_link"
-    robot_namespace="${namespace}"
-    suffix="back_right">
-    <origin xyz="-${sqrt2by2 * arm_length } -${sqrt2by2 * arm_length} ${motor_offset_top}" rpy="1.570796327 0 0"/>
-  </xacro:vertical_motor>
 </robot>

File: rotors_description/urdf/firefly_base.xacro (robot description, xacro)
@@ -29,5 +29,6 @@
   </xacro:if>
   <!-- Mount an ADIS16448 IMU. -->
-  <xacro:default_imu namespace="${namespace}" parent_link="${namespace}/base_link" />
+ <!--  <xacro:default_imu namespace="${namespace}" parent_link="${namespace}/base_link" /> -->
+ <xacro:edrone_odometry namespace="${namespace}" parent_link="${namespace}/base_link" />
   <xacro:if value="$(arg enable_ground_truth)">
     <xacro:ground_truth_imu_and_odometry namespace="${namespace}" parent_link="${namespace}/base_link" />

Commit message: arm_length of edrone_big changed to its actual value

File: rotors_description/urdf/crazyflie2.xacro (robot description, xacro)
@@ -35,5 +35,5 @@
   <xacro:property name="max_rot_velocity" value="2618" /> <!-- [rad/s] -->
   <xacro:property name="rotor_drag_coefficient" value="8.06428e-05" />
-   <xacro:property name="sqrt2by2" value="0.707106781186" />
+  <xacro:property name="sqrt2by2" value="0.707106781186" />
   <xacro:property name="rolling_moment_coefficient" value="0.000001" />
   <!-- Property Blocks -->

File: rotors_description/urdf/edrone_big.xacro (robot description, xacro)
@@ -10,5 +10,5 @@
   <xacro:property name="body_height" value="0.16" /> <!-- [m] -->
   <xacro:property name="mass_rotor" value="0.005" /> <!-- [kg] -->
-  <xacro:property name="arm_length" value="0.09" /> <!-- [m] -->
+  <xacro:property name="arm_length" value="0.18" /> <!-- [m] -->
   <!-- changed from 0.023 to 0.027 -->
   <xacro:property name="rotor_offset_top" value="0.0420" /> <!-- [m] -->
@@ -19,8 +19,9 @@
   <xacro:property name="time_constant_down" value="0.025" /> <!-- [s] -->
   <xacro:property name="max_rot_velocity" value="838" /> <!-- [rad/s] -->
-    <xacro:property name="motor_offset_top" value="-0.0409" />
+  <xacro:property name="motor_offset_top" value="-0.0409" />
   <xacro:property name="sin30" value="0.5" />
   <xacro:property name="cos30" value="0.866025403784" />
-  <xacro:property name="sqrt2" value="1.4142135623730951" />
+  <!-- <xacro:property name="sqrt2" value="1.4142135623730951" /> -->
+  <xacro:property name="sqrt2by2" value="0.707106781186" />
   <xacro:property name="rotor_drag_coefficient" value="8.06428e-05" />
   <xacro:property name="rolling_moment_coefficient" value="0.000001" />
@@ -65,5 +66,5 @@
     use_own_mesh="false"
     mesh="">
-    <origin xyz="${sqrt2 * arm_length} -${sqrt2 * arm_length} ${rotor_offset_top}" rpy="0 0 0" />
+    <origin xyz="${sqrt2by2 * arm_length} -${sqrt2by2 * arm_length} ${rotor_offset_top}" rpy="0 0 0" />
     <xacro:insert_block name="rotor_inertia" />
   </xacro:vertical_rotor>
@@ -74,5 +75,5 @@
     robot_namespace="${namespace}"
     suffix="front_right">
-    <origin xyz="${sqrt2 * arm_length} -${sqrt2 * arm_length} ${motor_offset_top}" rpy="1.570796327 0 0"/>
+    <origin xyz="${sqrt2by2 * arm_length} -${sqrt2by2 * arm_length} ${motor_offset_top}" rpy="1.570796327 0 0"/>
   </xacro:vertical_motor>
   <xacro:vertical_rotor
@@ -94,5 +95,5 @@
     use_own_mesh="false"
     mesh="">
-    <origin xyz="-${sqrt2 * arm_length} ${sqrt2 * arm_length} ${rotor_offset_top}" rpy="0 0 0" />
+    <origin xyz="-${sqrt2by2 * arm_length} ${sqrt2by2 * arm_length} ${rotor_offset_top}" rpy="0 0 0" />
     <xacro:insert_block name="rotor_inertia" />
   </xacro:vertical_rotor>
@@ -103,5 +104,5 @@
     robot_namespace="${namespace}"
     suffix="back_left">
-    <origin xyz="-${sqrt2 * arm_length} ${sqrt2 * arm_length} ${motor_offset_top}" rpy="1.570796327 0 0"/>
+    <origin xyz="-${sqrt2by2 * arm_length} ${sqrt2by2 * arm_length} ${motor_offset_top}" rpy="1.570796327 0 0"/>
   </xacro:vertical_motor>
   <xacro:vertical_rotor robot_namespace="${namespace}"
@@ -122,5 +123,5 @@
     use_own_mesh="false"
     mesh="">
-    <origin xyz="${sqrt2 * arm_length} ${sqrt2 * arm_length} ${rotor_offset_top}" rpy="0 0 0" />
+    <origin xyz="${sqrt2by2 * arm_length} ${sqrt2by2 * arm_length} ${rotor_offset_top}" rpy="0 0 0" />
     <xacro:insert_block name="rotor_inertia" />
   </xacro:vertical_rotor>
@@ -131,5 +132,5 @@
     robot_namespace="${namespace}"
     suffix="front_left">
-    <origin xyz="${sqrt2 * arm_length} ${sqrt2 * arm_length} ${motor_offset_top}" rpy="1.570796327 0 0"/>
+    <origin xyz="${sqrt2by2 * arm_length} ${sqrt2by2 * arm_length} ${motor_offset_top}" rpy="1.570796327 0 0"/>
   </xacro:vertical_motor>
   <xacro:vertical_rotor robot_namespace="${namespace}"
@@ -150,5 +151,5 @@
     use_own_mesh="false"
     mesh="">
-    <origin xyz="-${sqrt2 * arm_length} -${sqrt2 * arm_length} ${rotor_offset_top}" rpy="0 0 0" />
+    <origin xyz="-${sqrt2by2 * arm_length} -${sqrt2by2 * arm_length} ${rotor_offset_top}" rpy="0 0 0" />
     <xacro:insert_block name="rotor_inertia" />
   </xacro:vertical_rotor>
@@ -159,5 +160,5 @@
     robot_namespace="${namespace}"
     suffix="back_right">
-    <origin xyz="-${sqrt2 * arm_length} -${sqrt2 * arm_length} ${motor_offset_top}" rpy="1.570796327 0 0"/>
+    <origin xyz="-${sqrt2by2 * arm_length} -${sqrt2by2 * arm_length} ${motor_offset_top}" rpy="1.570796327 0 0"/>
   </xacro:vertical_motor>
 </robot>
